File: controller/pcb/usb_and_cp2102.sch (KiCad schematic (older format))
At the start: 14 parts, among them P1 USB_C_Plug_USB2.0, Q5 BC817, Q6 BC817, U3 LM1117-3.3, U4 CP2102N-A02-GQFN24

Commit message: wip qnfp28
Parts:
- removed S4: PWR, Connector_JST:JST_XH_B2B-XH-AM_1x02_P2.50mm_Vertical, symbol Connector_Generic:Conn_01x02
- removed U4: CP2102N-A02-GQFN24, cp2102:Silicon_Labs-CP2102N-A02-GQFN24-IPC_A, symbol terrarium-rescue:CP2102N-A02-GQFN24-CP2102N-A02-GQFN24
- added U4: CP2102N-A02-GQFN28, cp2102:Silicon_Labs-CP2102N-A02-GQFN28-IPC_A, symbol CP2102N-A02-GQFN28:CP2102N-A02-GQFN28
Connections:
- wire segments 62 -> 67
- no-connect marks 14 -> 18
Other:
- moved on the sheet: C4, C6, Q5, Q6, R19, R20
