File: controller/pcb/sensors.sch (KiCad schematic (older format))
At the start: 10 parts, among them Q4 S8050

Commit message: feat: add 5 pin sensor connectors
Parts:
- SENS0: renamed from SENS1; footprint Connector_JST:JST_XH_B3B-XH-AM_1x03_P2.50mm_Vertical -> Connector_JST:JST_XH_B5B-XH-AM_1x05_P2.50mm_Vertical; symbol Connector_Generic_MountingPin:Conn_01x03_MountingPin -> Connector_Generic:Conn_01x05
- SENS1: renamed from SENS2; footprint Connector_JST:JST_XH_B3B-XH-AM_1x03_P2.50mm_Vertical -> Connector_JST:JST_XH_B5B-XH-AM_1x05_P2.50mm_Vertical; symbol Connector_Generic_MountingPin:Conn_01x03_MountingPin -> Connector_Generic:Conn_01x05
- SENS2: renamed from SENS3; footprint Connector_JST:JST_XH_B3B-XH-AM_1x03_P2.50mm_Vertical -> Connector_JST:JST_XH_B5B-XH-AM_1x05_P2.50mm_Vertical; symbol Connector_Generic_MountingPin:Conn_01x03_MountingPin -> Connector_Generic:Conn_01x05
- SENS3: renamed from SENS4; footprint Connector_JST:JST_XH_B3B-XH-AM_1x03_P2.50mm_Vertical -> Connector_JST:JST_XH_B5B-XH-AM_1x05_P2.50mm_Vertical; symbol Connector_Generic_MountingPin:Conn_01x03_MountingPin -> Connector_Generic:Conn_01x05
- SENS4: renamed from SENS5; value 4 -> 5; footprint Connector_JST:JST_XH_B3B-XH-AM_1x03_P2.50mm_Vertical -> Connector_JST:JST_XH_B5B-XH-AM_1x05_P2.50mm_Vertical; symbol Connector_Generic_MountingPin:Conn_01x03_MountingPin -> Connector_Generic:Conn_01x05
- SENS5: renamed from SENS6; value 4 -> 6; footprint Connector_JST:JST_XH_B3B-XH-AM_1x03_P2.50mm_Vertical -> Connector_JST:JST_XH_B5B-XH-AM_1x05_P2.50mm_Vertical; symbol Connector_Generic_MountingPin:Conn_01x03_MountingPin -> Connector_Generic:Conn_01x05
Connections:
- net labels added: SCL_0, SCL_1, SCL_2, SCL_3, SCL_4, SCL_5, SDA_0, SDA_1, SDA_2, SDA_3, SDA_4, SDA_5
- wire segments 45 -> 44
- no-connect marks 6 -> 0
Other:
- moved on the sheet: LED5, Q4, R10, R17

Commit message: improved silk screen, tracing
Parts:
- SENS0, SENS1, SENS2, SENS5: footprint Connector_JST:JST_XH_B5B-XH-AM_1x05_P2.50mm_Vertical -> Connector_JST:JST_XH_B5B-XH-A_1x05_P2.50mm_Vertical
- SENS4: footprint Connector_JST:JST_XH_B5B-XH-AM_1x05_P2.50mm_Vertical -> Connector_JST:JST_XH_B6B-XH-AM_1x06_P2.50mm_Vertical
Changed lines of the file:
@@
 F 0 "SENS2" H 3150 2100 50  0000 L CNN
 F 1 "3" H 3400 1800 50  0000 L CNN
-F 2 "Connector_JST:JST_XH_B5B-XH-AM_1x05_P2.50mm_Vertical" H 3350 1800 50  0001 C CNN
+F 2 "Connector_JST:JST_XH_B5B-XH-A_1x05_P2.50mm_Vertical" H 3350 1800 50  0001 C CNN
 F 3 "~" H 3350 1800 50  0001 C CNN
 	1    3350 1800
@@
 F 0 "SENS0" H 1750 2100 50  0000 L CNN
 F 1 "1" H 2000 1800 50  0000 L CNN
-F 2 "Connector_JST:JST_XH_B5B-XH-AM_1x05_P2.50mm_Vertical" H 1950 1800 50  0001 C CNN
+F 2 "Connector_JST:JST_XH_B5B-XH-A_1x05_P2.50mm_Vertical" H 1950 1800 50  0001 C CNN
 F 3 "~" H 1950 1800 50  0001 C CNN
 	1    1950 1800
@@
 F 0 "SENS4" H 4450 2100 50  0000 L CNN
 F 1 "5" H 4700 1800 50  0000 L CNN
-F 2 "Connector_JST:JST_XH_B5B-XH-AM_1x05_P2.50mm_Vertical" H 4650 1800 50  0001 C CNN
+F 2 "Connector_JST:JST_XH_B6B-XH-AM_1x06_P2.50mm_Vertical" H 4650 1800 50  0001 C CNN
 F 3 "~" H 4650 1800 50  0001 C CNN
 	1    4650 1800
@@
 F 0 "SENS5" H 5300 2100 50  0000 L CNN
 F 1 "6" H 5400 1800 50  0000 L CNN
-F 2 "Connector_JST:JST_XH_B5B-XH-AM_1x05_P2.50mm_Vertical" H 5350 1800 50  0001 C CNN
+F 2 "Connector_JST:JST_XH_B5B-XH-A_1x05_P2.50mm_Vertical" H 5350 1800 50  0001 C CNN
 F 3 "~" H 5350 1800 50  0001 C CNN
 	1    5350 1800
@@
 F 0 "SENS1" H 2450 2100 50  0000 L CNN
 F 1 "2" H 2700 1800 50  0000 L CNN
-F 2 "Connector_JST:JST_XH_B5B-XH-AM_1x05_P2.50mm_Vertical" H 2650 1800 50  0001 C CNN
+F 2 "Connector_JST:JST_XH_B5B-XH-A_1x05_P2.50mm_Vertical" H 2650 1800 50  0001 C CNN
 F 3 "~" H 2650 1800 50  0001 C CNN
 	1    2650 1800
